File: rosa.kicad_pcb (KiCad board)
At the start: 2 copper layers, 284.8 x 94.3 mm, 145 parts, among them J1 Conn_01x04, SW1 SW_Push, U1 ATmega32U4-MU, Y1 16MHz

Commit message: add pcb art
Parts:
- added LOGO1: O-LOGO, board_logos:MY-LOGO-SVG, F.Cu at (165.1, 85.7)
- added LOGO2: O-LOGO, board_logos:oggi-logo, F.Cu at (177.0, 85.7)
Other:
- board text added: "+"
- board text added: "-"
- board text added: "ROSA60 PCB BY ILLUSION"

Commit message: routing tune up. finalize edge cuts, pcb art, and designator silkscreen. update git ignore.
Routing:
- net Row4: track 319.7 -> 320.5 mm
- net GND: vias 11 -> 4
Other:
- board size 284.8 x 94.3 mm -> 284.3 x 94.5 mm
- board text added: "ROSA PCB BY ILLUSION"
- board text removed: "ROSA60 PCB BY ILLUSION"

Commit message: change caps lock indicator R value
Parts:
- R5: value 1k -> 470
