File: rosa.sch (KiCad schematic (older format))
At the start: 145 parts

Commit message: finish routing
Parts:
- removed MX?: MX-NoLED, symbol MX_Alps_Hybrid:MX-NoLED
- added MX15: MX-NoLED, MX_Only:MXOnly-1U-NoLED, symbol MX_Alps_Hybrid:MX-NoLED
- C1, C2, C3, C4, C5, C6, C7, C8: renamed from C?; footprint (none) -> Capacitor_SMD:C_0603_1608Metric
- F1: renamed from F?; footprint (none) -> Fuse:Fuse_1206_3216Metric
- J1: renamed from J?; footprint (none) -> random-keyboard-parts:JST-SR-4
- MX1, MX10, MX11, MX12, MX13, MX16, MX18, MX19, MX2, MX20, MX21, MX22, MX23, MX24, MX25, MX26, MX27, MX28, MX29, MX3, MX33, MX34, MX35, MX36, MX37, MX38, MX39, MX4, MX40, MX41, MX42, MX43, MX46, MX47, MX48, MX49, MX5, MX50, MX51, MX52, MX53, MX54, MX55, MX58, MX6, MX60, MX64, MX7, MX8, MX9: renamed from MX?; footprint (none) -> MX_Only:MXOnly-1U-NoLED
- MX14: renamed from MX?; footprint (none) -> MX_Only:MXOnly-2U-NoLED
- MX17, MX30, MX59, MX61, MX63, MX65: renamed from MX?; footprint (none) -> MX_Only:MXOnly-1.5U-NoLED
- MX31: renamed from MX?; footprint (none) -> MX_Only:MXOnly-1.25U-FLIPPED
- MX32: renamed from MX?; footprint (none) -> MX_Only:MXOnly-1.75U
- MX44: renamed from MX?; footprint (none) -> MX_Only:MXOnly-2.25U-ReversedStabilizers-NoLED
- MX45: renamed from MX?; footprint (none) -> MX_Only:MXOnly-2.25U-NoLED
- MX56: renamed from MX?; footprint (none) -> MX_Only:MXOnly-1.75U-NoLED
- MX57: renamed from MX?; footprint (none) -> MX_Only:MXOnly-2.75U-NoLED
- MX62: renamed from MX?; footprint (none) -> MX_Only:MXOnly-7U-ReversedStabilizers-NoLED
- R1, R2, R3, R4: renamed from R?; footprint (none) -> Resistor_SMD:R_0603_1608Metric
- SW1: renamed from SW?; footprint (none) -> footprints-and-logos:K2-1187SQ-A4SW-06
- Y1: renamed from Y?; footprint (none) -> Crystal:Crystal_SMD_3225-4Pin_3.2x2.5mm
- gave numbers to parts that had none: 64
Connections:
- net labels added: Col0, Col1, Col10, Col11, Col12, Col13, Col2, Col3, Col4, Col5, Col6, Col7, Col8, Col9, D1+, D1-, Row0, Row1, Row2, Row3, Row4, VCC
- wire segments 315 -> 327
Other:
- moved on the sheet: C1, C2, C3, C4, C5, C6, C7, C8, D1, D10, D11, D12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

Commit message: add pcb art
Parts:
- added LOGO1: O-LOGO, board_logos:MY-LOGO-SVG, symbol logos:O-LOGO
- added LOGO2: O-LOGO, board_logos:oggi-logo, symbol logos:O-LOGO
Changed lines of the file:
@@
 Text GLabel 13950 1500 2    50   Input ~ 0
 Row3
+$Comp
+L logos:O-LOGO LOGO1
+U 1 1 6058DB7E
+P 13700 11950
+F 0 "LOGO1" H 13874 11996 50  0000 L CNN
+F 1 "O-LOGO" H 13874 11905 50  0000 L CNN
+F 2 "board_logos:MY-LOGO-SVG" H 13700 11950 50  0001 C CNN
+F 3 "" H 13700 11950 50  0001 C CNN
+	1    13700 11950
+	1    0    0    -1
+$EndComp
+$Comp
+L logos:O-LOGO LOGO2
+U 1 1 60638FCB
+P 14400 11950
+F 0 "LOGO2" H 14574 11996 50  0000 L CNN
+F 1 "O-LOGO" H 14574 11905 50  0000 L CNN
+F 2 "board_logos:oggi-logo" H 14400 11950 50  0001 C CNN
+F 3 "" H 14400 11950 50  0001 C CNN
+	1    14400 11950
+	1    0    0    -1
+$EndComp
 $EndSCHEMATC

Commit message: change caps lock indicator R value
Parts:
- R5: value 1k -> 470
Changed lines of the file:
@@
 P 4850 10000
 F 0 "R5" H 4950 10000 50  0000 C CNN
-F 1 "1k" H 4950 10100 50  0000 C CNN
+F 1 "470" H 4950 10100 50  0000 C CNN
 F 2 "Resistor_SMD:R_0603_1608Metric" H 4850 10000 50  0001 C CNN
 F 3 "~" H 4850 10000 50  0001 C CNN
